File: hardware/kicad/inputs.kicad_sch (KiCad schematic)
At the start: 0 parts

Commit message: input circuitry
Parts:
- added C1: 68pF, symbol Device:C
- added C2: 100nF, symbol Device:C
- added C3, C4: 6.2nF, Package_DIP:DIP-24_W7.62mm, symbol Device:C
- added C5, C6: 47uF, symbol Device:C
- added D1: D_TVS, Diode_SMD:D_SOD-323, symbol Device:D_TVS
- added D2, D3: D_TVS, Diode_SMD:D_SMA, symbol Device:D_TVS
- added J1: XLR3_AudioJack2_Combo, symbol Connector_Audio:XLR3_AudioJack2_Combo
- added R1: 200, symbol Device:R
- added R2: 1M, symbol Device:R
- added R3, R4: 100, symbol Device:R
- added R5, R6: 2.2k, symbol Device:R
Connections:
- new net: C3.1, C6.1, R4.2
- new net: C6.2, R6.2
- new net: C1.1, C2.1, R1.2
- new net: C2.2, R2.2
- new net: C4.2, C5.1, R3.2
- new net: C5.2, R5.2
- new net SHIELD_GND: C3.2, C4.1, D2.2 (A2), D3.1 (A1), J1.1
- new net TS1_IN: D1.1 (A1), J1.T, R1.1
- new net TS1_SLVE: C1.2, D1.2 (A2), J1.S
- new net VBIAS: R2.1, R5.1, R6.1
- new net XLR1_N: D3.2 (A2), J1.3, R3.1
- new net XLR1_P: D2.1 (A1), J1.2, R4.1
Other:
- note added: "2.2k bias resistor matches microphone Z - Rbias = 10(Z_mic) = 10(200) = ~2.2k"
- note added: "47uF is large enough to block the 48V DC Phantom Power fc =~ 1.47Hz, audible signals are unaffected"
- note added: "C_SHUNT = 1 / (2pi * Req * fc) target fc is 125 KHz ish C_SHUNT = 1 / (2pi * 200 * 125000) =~ 6.2nF"
- note added: "R_SERIES = 100 ; HF standard"
- note added: "TVS rated with V_RWM = 58V, provides solid headroom for phantom power - higher-capacitance adds to RC filter"
- note added: "TVS rated with V_RWM = 8V, prevents solid headroom for audio voltages - clamps @ 18.5 V, a bit steep but it was the best available option - low-capacitance @ 1MHz of 3pF"
- note added: "VBIAS = VCC/2 (1.65)| voltage divider + buffer"
- note added: "coupling capacitor used to pass AC while blocking DC. 100nF sets f_c =~ 1.6Hz which passes all instrument/line-level freqs. 1M ohm is a standard bias resistor value."
- note added: "instrument audio impedance is typically ~10-50k Ω R should be small, sig. less than our audio impedance R = 200. cutoff target frequency is 50kHz. C = 1 / (2pi * fc * (Rins + R) C = 1 / (2pi * 50000 * 50200) =~ 63.4 pF"
- company: (none) -> Jeevan Sanchez
- title: (none) -> Audio Inputs

Commit message: usb interface
Parts:
- added C10, C13, C16, C7: 6.2nF, Package_DIP:DIP-24_W7.62mm, symbol Device:C
- added C11, C17: 100nF, symbol Device:C
- added C12, C18: 68pF, symbol Device:C
- added C14, C15, C8, C9: 47uF, symbol Device:C
- added D10: 1N4148, Diode_THT:D_DO-35_SOD27_P7.62mm_Horizontal, symbol Diode:1N4148
- added D4, D5, D7, D8: D_TVS, Diode_SMD:D_SMA, symbol Device:D_TVS
- added D6, D9: D_TVS, Diode_SMD:D_SOD-323, symbol Device:D_TVS
- added J2, J3: XLR3_AudioJack2_Combo, symbol Connector_Audio:XLR3_AudioJack2_Combo
- added K1: G6K-2, Relay_THT:Relay_SPDT_Omron_G6E, symbol Relay:G6K-2
- added Q1: 2N7002, Package_TO_SOT_SMD:SOT-23, symbol Transistor_FET:2N7002
- added R10, R14, R16, R18, R22, R24: 2.2k, symbol Device:R
- added R11, R12, R19, R20: 100, symbol Device:R
- added R13, R17, R21, R7, R8, R9: 6.8k, symbol Device:R
- added R15, R27: 1M, symbol Device:R
- added R23: 100, Package_TO_SOT_SMD:SOT-23, symbol Device:R
- added R25: 100k, Package_TO_SOT_SMD:SOT-23, symbol Device:R
- added R28: 15k, symbol Device:R
- added R29: 3.3k, symbol Device:R
- added R34, R35, R36, R37, R38, R39: 100k, symbol Device:R
- R1: value 200 -> 2.2k
Connections:
- net SHIELD_GND: now also C10.2, C13.1, C16.2, C7.1, D4.1 (A1), D5.2 (A2), D7.1 (A1), D8.2 (A2), J2.1, J3.1
- net VBIAS: now also R10.1, R14.1, R15.1, R18.1, R22.1, R27.1
- net at C3.1, C6.1, R4.2: now also R8.2
- net AFE1_INN: now reaches C6.2, R6.2
- net AFE1_INN: now also R37.2
- net at C4.2, C5.1, R3.2: now also R7.2
- net AFE1_INP: now reaches C5.2, R5.2
- net AFE1_INP: now also R36.2
- new net: C10.1, C9.1, R12.2, R13.2
- new net: C15.1, C16.1, R20.2, R21.2
- new net: Q1.1 (G), R23.2
- new net: D10.2 (A), K1.8, Q1.3 (D)
- new net: C17.2, R27.2
- new net: C13.2, C14.1, R17.2, R19.2
- new net: C7.2, C8.1, R11.2, R9.2
- new net: C17.1, C18.1, R24.2
- new net: C11.1, C12.1, R16.2
- new net: C11.2, R15.2
- new net: K1.6, R29.2
- new net +5V: D10.1 (K), K1.1
- new net AFE2_INN: C9.2, R14.2, R38.2
- new net AFE2_INP: C8.2, R10.2, R39.2
- new net AFE3_INN: C15.2, R22.2, R35.2
- new net AFE3_INP: C14.2, R18.2, R34.2
- new net AGND: R34.1, R35.1, R36.1, R37.1, R38.1, R39.1
- new net GND: Q1.2 (S), R25.1, R29.1
- new net HIZ_FET_GATE: R23.1, R25.2
- new net PHANTOM_48V: R13.1, R17.1, R21.1, R7.1, R8.1, R9.1
- new net TS2_IN: D6.1 (A1), J2.T, R16.1
- new net TS2_SLVE: C12.2, D6.2 (A2), J2.S
- new net TS3_HIZ_OUT: D9.1 (A1), K1.2, K1.5, R24.1, R28.1
- new net TS3_IN: J3.T, K1.3, R28.2
- new net TS3_SLVE: C18.2, D9.2 (A2), J3.S
- new net XLR2_N: D4.2 (A2), J2.3, R11.1
- new net XLR2_P: D5.1 (A1), J2.2, R12.1
- new net XLR3_N: D7.2 (A2), J3.3, R19.1
- new net XLR3_P: D8.1 (A1), J3.2, R20.1
- no-connect marks 0 -> 2
Other:
- note added: "* J3 feautres hi-z switching"
- note added: "*cleaned 48V"
- note added: "DPDT relay to provide unattentuated HI-Z instrument input by default, while switching in a 15k/3.3k voltage divider pad (-14.9dB) for line-level signals when energized."
- note added: "INST/LINE Switch"
- note added: "instrument audio impedance is typically ~10-50k Ω R1 is in series with the 1M bias, so loading is R1/1M. R1 limits TVS residual clamp current to ≤10 mA: R1 ≥ (18.5 − 3.3 − 0.3) / 10 mA ≈ 1.5k → use 2.2k. cutoff target frequency is 50kHz. C = 1 / (2pi * fc * (Rins + R) C = 1 / (2pi * 50000 * 50200) =~ 63.4 pF"
- note added: "minimize loss. loss = 20log_10(R_L/( R_L + R_bias)) with R_bias = 10k, R_L = 20k loss = -0.17 dB"
- note added: "minimize loss. loss = 20log_10(R_L/( R_L + R_bias)) with R_bias = 1M, R_L = 50k loss = -0.09 dB"
- note removed: "2.2k bias resistor matches microphone Z - Rbias = 10(Z_mic) = 10(200) = ~2.2k"
- note removed: "VBIAS = VCC/2 (1.65)| voltage divider + buffer"
- note removed: "instrument audio impedance is typically ~10-50k Ω R should be small, sig. less than our audio impedance R = 200. cutoff target frequency is 50kHz. C = 1 / (2pi * fc * (Rins + R) C = 1 / (2pi * 50000 * 50200) =~ 63.4 pF"
- moved on the sheet: C1, C2, C3, C4, D1, D2, D3, J1A, J1B, R1, R2, R3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
