File: hardware/kicad/mcu.kicad_sch (KiCad schematic)
At the start: 0 parts

Commit message: stm32h723 breakout
Parts:
- added C21, C29: 10uF, Package_QFP:LQFP-100_14x14mm_P0.5mm, symbol Device:C
- added C22, C23, C24, C25, C26, C27, C28, C32, C34: 100nF, Package_QFP:LQFP-100_14x14mm_P0.5mm, symbol Device:C
- added C30, C31: 2.2uF, Package_QFP:LQFP-100_14x14mm_P0.5mm, symbol Device:C
- added C33: 1uF, Package_QFP:LQFP-100_14x14mm_P0.5mm, symbol Device:C
- added C36, C37: 10pF, Package_QFP:LQFP-100_14x14mm_P0.5mm, symbol Device:C
- added D16: DEBUG_LED, ESD122DMYR:DIO_ESD122DMYR, symbol Device:LED
- added D17: HBEAT_LED, ESD122DMYR:DIO_ESD122DMYR, symbol Device:LED
- added D18, D19, D20, D21, D22, D23, D24, D25, D26, D27, D28: LED, ESD122DMYR:DIO_ESD122DMYR, symbol Device:LED
- added FB1: FerriteBead, symbol Device:FerriteBead
- added R40: 10k, symbol Device:R
- added R41, R42, R44, R45, R46, R47: 100, symbol Device:R
- added SW3: SW_NRST, Button_Switch_SMD:Nidec_Copal_CAS-120A, symbol Switch:SW_Push
- added SW4: SW_BOOT0, Button_Switch_SMD:Nidec_Copal_CAS-120A, symbol Switch:SW_Push
- added U1: STM32H723VETx, Package_QFP:LQFP-100_14x14mm_P0.5mm, symbol MCU_ST_STM32H7:STM32H723VETx
- added Y1: SYS_OSC, symbol Device:Crystal
Connections:
- new net: C37.2, U1.13 (PH1), Y1.2
- new net: D20.2 (A), D21.1 (K), D22.1 (K), D22.2 (A), D23.1 (K), D23.2 (A), D24.2 (A), D25.1 (K), D26.2 (A), D27.1 (K), D28.2 (A), R46.2, R47.2
- new net: R44.1, U1.51 (PB12)
- new net: D18.1 (K), D19.2 (A), D26.1 (K), D27.2 (A), D28.1 (K), R44.2
- new net: C21.1, C22.1, C32.2, C33.2, FB1.2, U1.20 (VREF+), U1.21 (VDDA)
- new net: C31.2, U1.73 (VCAP)
- new net: D18.2 (A), D19.1 (K), D20.1 (K), D21.2 (A), D24.1 (K), D25.2 (A), R45.2
- new net: C36.2, U1.12 (PH0), Y1.1
- new net: D17.2 (A), R42.2
- new net: R46.1, U1.53 (PB14)
- new net: C30.2, U1.48 (VCAP)
- new net: R41.1, U1.63 (PC6)
- new net: D16.2 (A), R41.2
- new net: R45.1, U1.52 (PB13)
- new net: R42.1, U1.64 (PC7)
- new net: R47.1, U1.54 (PB15)
- new net +3.3V: C23.2, C24.2, C25.2, C26.2, C27.2, C28.2, C29.2, SW4.2, U1.100 (VDD), U1.11 (VDD), U1.27 (VDD), U1.50 (VDD), U1.6 (VBAT), U1.75 (VDD)
- new net +3.3VA_STM: FB1.1
- new net GND: C21.2, C22.2, C23.1, C24.1, C25.1, C26.1, C27.1, C28.1, C29.1, C30.1, C31.1, C32.1, C33.1, C34.1, C36.1, C37.1, D16.1 (K), D17.1 (K), R40.2, SW3.2, U1.10 (VSS), U1.19 (VSSA), U1.26 (VSS), U1.49 (VSS), U1.74 (VSS), U1.99 (VSS)
- new net STM_BOOT0: R40.1, SW4.1, U1.94 (BOOT0)
- new net STM_NRST: C34.2, SW3.1, U1.14 (NRST)
- new net SWDCLK: U1.76 (PA14(JTCK)
- new net SWDIO: U1.72 (PA13(JTMS)
- new net USB_N: U1.70 (PA11)
- new net USB_P: U1.71 (PA12)
- no-connect marks 0 -> 1
Other:
- note added: "100nF/VDD pin"
- note added: "CL = 8pF * use symmetry, (C1 = C2 = C), stray capictance CS =~ 3pF CL = C/2 + Cs C = 2(CL - CS) C = 2(8-3)= 10 pF"
- note added: "Charliplexed LED Matrix"
- note added: "R = (VS - VF) / I R = (3.3-2) / 0.02 = 65 ~ 100 ohm [amber]"
- note added: "R = (VS - VF) / I R = (3.3-3.1) / 0.02 = 10 ~ 100 ohm (SAFE) [white]"
- note added: "active low"
- note added: "internal pullup"
- company: (none) -> Jeevan Sanchez
- title: (none) -> STM32H723 Breakout Circuitry
Changed lines of the file:
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@@
 	(generator "eeschema")
 	(generator_version "10.0")
-	(paper "A4")
-)
+	(paper "A3")
+	(title_block
+		(title "STM32H723 Breakout Circuitry")
+		(company "Jeevan Sanchez")
+		(comment 1 "Vireo Lite")
+	)
