File: hardware/kicad/usb.kicad_sch (KiCad schematic)
At the start: 0 parts

Commit message: usb interface
Parts:
- added D12: USB_IN_LED, symbol Device:LED
- added D13: ESD122DMYR, ESD122DMYR:DIO_ESD122DMYR, symbol ESD122DMYR:ESD122DMYR
- added J4: USB_C_Receptacle_USB2.0_16P, Connector_USB:USB_C_Receptacle_GCT_USB4125-xx-x_6P_TopMnt_Horizontal, symbol Connector:USB_C_Receptacle_USB2.0_16P
- added R30, R31: 5.1k, symbol Device:R
- added R32: 200, symbol Device:R
Connections:
- new net: J4.A5 (CC1), R30.1
- new net: J4.B5 (CC2), R31.2
- new net: D12.2 (A), R32.2
- new net GND: D12.1 (K), D13.1, J4.A1 (GND), J4.A12 (GND), J4.A8 (SBU1), J4.B1 (GND), J4.B12 (GND), J4.B8 (SBU2), J4.SH (SHIELD), R30.2, R31.1
- new net USB_N: D13.3, J4.A7 (D-), J4.B7 (D-)
- new net USB_P: D13.2, J4.A6 (D+), J4.B6 (D+)
- new net VBUS_RAW: J4.A4 (VBUS), J4.A9 (VBUS), J4.B4 (VBUS), J4.B9 (VBUS), R32.1
Other:
- company: (none) -> Jeevan Sanchez
- title: (none) -> USB Interface

Commit message: stm32h723 breakout
Parts:
- added C35: 100nF, Package_QFP:LQFP-100_14x14mm_P0.5mm, symbol Device:C
- added D15: ESD122DMYR, ESD122DMYR:DIO_ESD122DMYR, symbol ESD122DMYR:ESD122DMYR
- added J5: SWD_HEADER, symbol Connector_Generic:Conn_01x04
Connections:
- net GND: now also C35.1, D15.1, J5.1 (Pin_1)
- new net SWDCLK: D15.3, J5.3 (Pin_3)
- new net SWDIO: D15.2, J5.2 (Pin_2)
- new net VSWD: C35.2, J5.4 (Pin_4)
Other:
- title: USB Interface -> Flash/Debug Interface
- moved on the sheet: D12, D13, J4, R30, R31, R32
